File: hardware/neoimage_sensors small.brd (EAGLE design)
At the start: 28.3 x 23.5 mm, 35 parts, among them J8 AUDIO_JACK_3.5MM, U1 LIS3DH, U2 LIGHT_SENSORALS, U4 STM32F030F4P6TR, U6 LMV358

Commit message: cleanup schematic, name signals, pdf
Parts:
- L1: value 3.3µH/±20%/450mA -> 1µH
Connections:
- net PA1 renamed LIGHT
- net PA10 renamed SCL
- net PA13 renamed SWDIO
- net PA14 renamed SWCLK
- net PA4 renamed AIN0
- net PA5 renamed AIN4
- net PA6 renamed AIN3
- net PA7 renamed AIN2
- net PA9 renamed SDA
- net PB1 renamed AIN1
Changed lines of the file:
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@@
 <attribute name="VALUE" x="11.3284" y="13.335" size="0.6096" layer="27" font="vector" rot="R90" align="top-center"/>
 </element>
-<element name="L1" library="SparkFun-Coils" library_urn="urn:adsk.eagle:library:512" package="0805" package3d_urn="urn:adsk.eagle:package:37579/1" value="3.3µH/±20%/450mA" x="22.86" y="12.192" smashed="yes">
+<element name="L1" library="SparkFun-Coils" library_urn="urn:adsk.eagle:library:512" package="0805" package3d_urn="urn:adsk.eagle:package:37579/1" value="1µH" x="22.86" y="12.192" smashed="yes">
 <attribute name="PROD_ID" value="NDUC-13076" x="16.764" y="-33.528" size="1.778" layer="27" display="off"/>
 </element>
@@
 <contactref element="J1" pad="7"/>
 </signal>
-<signal name="PA9">
+<signal name="SDA">
 <contactref element="U4" pad="17"/>
 <contactref element="R2" pad="2"/>
@@
 <wire x1="13.4874" y1="16.256" x2="14.5034" y2="15.24" width="0.1524" layer="1"/>
 </signal>
-<signal name="PA10">
+<signal name="SCL">
 <contactref element="U4" pad="18"/>
 <contactref element="R5" pad="2"/>
@@
 <wire x1="12.7908" y1="17.867" x2="12.2302" y2="17.867" width="0.1524" layer="1"/>
 </signal>
-<signal name="PA1">
+<signal name="LIGHT">
 <contactref element="U4" pad="7"/>
 <contactref element="R8" pad="2"/>
@@
 <wire x1="1.166" y1="0.916" x2="1.166" y2="0.7128" width="0.1524" layer="1"/>
 </signal>
-<signal name="PA4">
+<signal name="AIN0">
 <contactref element="U4" pad="10"/>
 <contactref element="J3" pad="1"/>
@@
 <wire x1="6.0932" y1="22.8572" x2="3.556" y2="20.32" width="0.1524" layer="1"/>
 </signal>
-<signal name="PA5">
+<signal name="AIN4">
 <contactref element="U4" pad="11"/>
 <contactref element="J3" pad="5"/>
@@
 <wire x1="9.197" y1="22.352" x2="11.176" y2="22.352" width="0.1524" layer="16"/>
 </signal>
-<signal name="PA6">
+<signal name="AIN3">
 <contactref element="U4" pad="12"/>
 <contactref element="J3" pad="4"/>
@@
 <wire x1="13.589" y1="22.098" x2="13.258" y2="21.767" width="0.1524" layer="1"/>
 </signal>
-<signal name="PA7">
+<signal name="AIN2">
 <contactref element="U4" pad="13"/>
 <contactref element="J3" pad="3"/>
@@
 <wire x1="13.716" y1="21.463" x2="13.37" y2="21.117" width="0.1524" layer="1"/>
 </signal>
-<signal name="PB1">
+<signal name="AIN1">
 <contactref element="U4" pad="14"/>
 <contactref element="J3" pad="2"/>
@@
 <wire x1="21.717" y1="21.209" x2="23.368" y2="21.209" width="0.1524" layer="16"/>
 </signal>
-<signal name="PA13">
+<signal name="SWDIO">
 <contactref element="U4" pad="19"/>
 <contactref element="D" pad="TP"/>
@@
 <wire x1="11.176" y1="17.2664" x2="11.689365625" y2="17.779765625" width="0.1524" layer="16"/>
 </signal>
-<signal name="PA14">
+<signal name="SWCLK">
 <contactref element="U4" pad="20"/>
 <contactref element="C" pad="TP"/>
